Commit message: added rplidar in drone definition

File: models/aerotrain/aerotrain.urdf (robot description, URDF)
Before this commit: robot aerotrain, 10 links, 9 joints
Links:
- added link rplidar_link, mass 0.015; visual cylinder length=0.002 radius=0.01
Joints:
- added joint rplidar_joint: type fixed, parent base_link, child rplidar_link, origin xyz=0.0  0  0.05 rpy=0 0 0, axis 0 0 0, limit lower=0 upper=0 effort=0 velocity=0
